File: CP2102N_bb.kicad_pcb (KiCad board)
At the start: 2 copper layers, 18.4 x 20.3 mm, 18 parts, among them J1 USB_B_Micro, J2 UART, J3 Other, J4 Other, U1 CP2102N

Commit message: Update project to use a local version of the hand-solderable QFP-24 footprint.
Parts:
- U1: footprint custom_footprints:QFN-24-1EP_4x4mm_HandSolder -> CP2102N_bb:QFN-24-1EP_4x4mm_HandSolder
